File: Rev 3/PCB ESP32 S3 Wroom 1 n16r8/PCB ESP32 S3 Wroom 1 n16r8.kicad_sch (KiCad schematic)
At the start: 36 parts, among them IC1 LM2675N-3.3_NOPB, J1 AudioJack3_SwitchT, M1 Haptic Feedback, Q1 BS170, SW1 Home, SW2 Back, SW3 Play/Pause, SW4 Power, SW5 Menu, SW6 Hold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

Commit message: updated inductor footprint
to be a standard 2424 (6060 metric) mount for a power rectifier.
Parts:
- L1: footprint Capacitor_SMD:C_0603_1608Metric -> Inductor_SMD:L_Coilcraft_XAL6060-XXX
Changed lines of the file:
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@@
 			)
 		)
-		(property "Footprint" "Capacitor_SMD:C_0603_1608Metric"
+		(property "Footprint" "Inductor_SMD:L_Coilcraft_XAL6060-XXX"
 			(at 115.57 73.66 0)
 			(effects

Commit message: changed out power regulator
- JLCPCB part package sizes
- new chip supports 4.5v-36v so it will work with usb power
Parts:
- removed D2: 1A, 40 V Schottky rectifier, Diode_SMD:D_SOD-323_HandSoldering, symbol Diode:SB120
- removed IC1: LM2675N-3.3_NOPB, LM2675-3.3:DIP794W53P254L959H508Q8N, symbol LM2675N-3_3_NOPB:LM2675N-3.3_NOPB
- added R14: 69.8K, Resistor_SMD:R_01005_0402Metric, symbol Device:R
- added R15: 22.1K, Resistor_SMD:R_01005_0402Metric, symbol Device:R
- added U1: LMR54410DBVR, LMR54410DBVR:SOT95P280X145-6N, symbol LMR54410DBVR:LMR54410DBVR
- C1: value 10 nF -> .1 uF; footprint Capacitor_SMD:C_2220_5750Metric -> Capacitor_SMD:C_0201_0603Metric
- C2: value 100 uF -> 2.2 uF; footprint Capacitor_SMD:C_2220_5750Metric -> Capacitor_SMD:C_0201_0603Metric
- C3: value 68uF -> 10uF; footprint Capacitor_SMD:C_2220_5750Metric -> Capacitor_SMD:C_0201_0603Metric
- L1: value 47uH -> 15uH; footprint Inductor_SMD:L_Coilcraft_XAL6060-XXX -> Inductor_SMD:L_Vishay_IFSC-1515AH_4x4x1.8mm
Connections:
- net 5V: now also U1.4 (EN), U1.5 (VIN)
- net GND: now also R15.1, U1.2 (GND)
- net VDD: now also R14.2
- net at C1.1, L1.2: now also U1.6 (SW)
- net at C1.2: now also U1.1 (CB)
- new net: R14.1, R15.2, U1.3 (FB)
Other:
- moved on the sheet: C1, C2

Commit message: updated pcb and fixed footprints
Parts:
- C1, C2, C3: footprint Capacitor_SMD:C_0201_0603Metric -> Capacitor_SMD:C_0603_1608Metric
- R14, R15: footprint Resistor_SMD:R_01005_0402Metric -> Resistor_SMD:R_01005_0402Metric_Pad0.57x0.30mm_HandSolder
Changed lines of the file:
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@@
 			)
 		)
-		(property "Footprint" "Capacitor_SMD:C_0201_0603Metric"
+		(property "Footprint" "Capacitor_SMD:C_0603_1608Metric"
 			(at 102.5652 85.09 0)
 			(effects
@@
 			)
 		)
-		(property "Footprint" "Capacitor_SMD:C_0201_0603Metric"
+		(property "Footprint" "Capacitor_SMD:C_0603_1608Metric"
 			(at 120.65 70.8152 0)
 			(effects
@@
 			)
 		)
-		(property "Footprint" "Resistor_SMD:R_01005_0402Metric"
+		(property "Footprint" "Resistor_SMD:R_01005_0402Metric_Pad0.57x0.30mm_HandSolder"
 			(at 97.028 87.63 90)
 			(effects
@@
 			)
 		)
-		(property "Footprint" "Resistor_SMD:R_01005_0402Metric"
+		(property "Footprint" "Resistor_SMD:R_01005_0402Metric_Pad0.57x0.30mm_HandSolder"
 			(at 97.028 95.25 90)
 			(effects
@@
 			)
 		)
-		(property "Footprint" "Capacitor_SMD:C_0201_0603Metric"
+		(property "Footprint" "Capacitor_SMD:C_0603_1608Metric"
 			(at 136.1948 88.9 0)
 			(effects
